File: standard_keyboard.sch (KiCad schematic (older format))
At the start: 12 parts

Commit message: update
Parts:
- added D1, D10, D11, D12, D13, D14, D15, D16, D17, D18, D19, D2, D20, D21, D22, D23, D24, D25, D3, D4, D5, D6, D7, D8, D9: D, My_Keyboard:D_SOD-123, symbol Device:D
- added SW1, SW10, SW11, SW12, SW13, SW14, SW15, SW16, SW17, SW18, SW19, SW2, SW20, SW21, SW22, SW23, SW24, SW25, SW3, SW4, SW5, SW6, SW7, SW8, SW9: SW_Push, My_Keyboard:XSwitch, symbol Switch:SW_Push
- C1, C2, C3, C4: renamed from C?; footprint (none) -> Capacitor_SMD:C_0603_1608Metric_Pad1.05x0.95mm_HandSolder
- J1: renamed from J?; footprint (none) -> Connector_USB:USB_Micro-B_Molex-105017-0001
- J2: renamed from J?; footprint (none) -> Connector_PinHeader_2.54mm:PinHeader_1x04_P2.54mm_Vertical
- R1, R2, R3: renamed from R?; footprint (none) -> Resistor_SMD:R_0603_1608Metric_Pad1.05x0.95mm_HandSolder
- SW26: renamed from SW?; footprint (none) -> My_Keyboard:1101VS-E
- gave numbers to parts that had none: 2
Connections:
- net labels added: COL0, COL1, COL2, COL3, COL4, ROW0, ROW1, ROW2, ROW3, ROW4, USB_D+, USB_D-
- net labels removed: USB_DM, USB_DP
- wire segments 36 -> 188
Other:
- moved on the sheet: U2
